File: ATA_Test.brd (EAGLE design)
At the start: 112.4 x 60.5 mm, 119 parts, among them IC2 LM833D, J1 SJ1-3523N, J2 A-2004-2-4-LPS-N-R, J3 SJ1-3523N, J4 SJ1-3523N, J5 SJ-2509N, Q1 MMBT3904, U1 PCM1681PWPR, U2 RASPBERRY_PICOTH, U3 TLV320ADC3140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

Commit message: adding pdf
Parts:
- added JP2: (no value), pinhead:1X02
- added Q2, Q3: DNP, ruark2:SOT23-3_CENTERED
- added Q4: MMBT3904, ruark2:SOT23-3_CENTERED
- added R39, R40, R41, R45: DNP, ruark2:0603
- added R46, R48, R55: 10, ruark2:0603
- added R54: 2k, ruark2:0603
- added R56: 10k, ruark2:0603
- C35, C46: value 1210_CAPACITOR -> 100uF
- C44, C49, C50, C51: value sel -> 0.1uF
- C45, C47: value sel -> 1nF
- R18: value 10 -> DNP
- R20: value 10 -> 1k
- R30: value sel -> DNP
- R31, R42, R43: value sel -> 1k
- R32, R44, R51: value sel -> 100
- R47, R52, R53: value sel -> 10k
- R49: value sel -> 10
- moved R18 9.01 mm to (73.9, 47.5), turned to 135 degrees
Connections:
- new net F/R_R: Q3.1, R21.1, R45.1, R48.1
- new net N$56: C11.2, R55.1
- new net N$58: Q4.1, R56.1
- new net RM_R: Q2.1, R34.1, R39.1, R46.1
- net ADC_IN1: now also R55.2; no longer C11.2
- net DAC_BCK: now also R18.1
- net DAC_SCK: now also R18.2
- net F/R: now also Q3.3, R41.2, R48.2; no longer R21.1
- net GND: now also JP2.2, Q2.2, Q3.2, Q4.2, R39.2, R45.2, R54.1
- net N$26: now also R54.2
- net N$28: now also JP2.1, Q4.3; no longer R18.1, U2.11
- net N$29: now also R56.2
- net RM: now also Q2.3, R40.2, R46.2; no longer R34.1
- net V+: now also R40.1, R41.1
Routing:
- net N$29: track 12.2 -> 65.0 mm
- net V+: track 48.9 -> 86.5 mm
- net F/R_R: track 0.00 -> 33.1 mm
- net RM_R: track 0.00 -> 27.5 mm
- net F/R: track 39.5 -> 13.9 mm
- net RM: track 40.0 -> 19.9 mm
- net GND: track 110.4 -> 117.6 mm, vias 66 -> 72
- net ADC_IN1: track 55.6 -> 51.6 mm
- net +5V: track 178.9 -> 181.4 mm
- net N$56: track 0.00 -> 2.38 mm
- net N$58: track 0.00 -> 1.89 mm
- net N$26: track 2.46 -> 4.27 mm
- net DAC_BCK: track 29.7 -> 30.9 mm
- net ADC_IN3: track 108.2 -> 108.8 mm
- net N$28: track 2.96 -> 2.41 mm
Other:
- board text added: "(GP1)"
- board text added: "OC"
- board text added: "OPEN COLLECTOR"
